Commit message: Add rplidar_ros package

File: models/skn_model.urdf (robot description, URDF)
Before this commit: robot skn_agv, 5 links, 4 joints
Links:
- added link laser; visual cylinder length=0.03 radius=0.03
- added link tower; visual cylinder length=0.58 radius=0.04
Joints:
- added joint tower_base_link_joint: type fixed, parent base_link, child tower, origin xyz=-0.09 0 0.29 rpy=0 0 0
- added joint tower_laser_joint: type fixed, parent tower, child laser, origin xyz=0 0 0.30 rpy=0 0 0
- joint left_wheel_upper_joint: type continuous -> fixed
- joint right_wheel_upper_joint: type continuous -> fixed
